File: microcard/infred.kicad_sch (KiCad schematic)
At the start: 19 parts, among them Q3 2N7002, Q5 BSS138PS,115, Q6 2N7002, U8 DYWH-IRM-H238T/2T

Commit message: semi-finished pcb, pages
Parts:
- renumbered C31 to C11, D6 to D4, LED1 to LED3, LED2 to LED4, LED3 to LED5, Q6 to Q4, Q3 to Q6, R33 to R26, R31 to R27, R23 to R28, R24 to R29, R25 to R30, R29 to R31, R26 to R32, R30 to R33, R32 to R34, U8 to U5
Changed lines of the file:
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@@
 		(on_board yes)
 		(dnp no)
-		(property "Reference" "C31"
+		(property "Reference" "C11"
 			(at 106.426 89.408 0)
 			(effects
@@
 			(project "microcard"
 				(path "/d4dbc2bb-914b-4f67-85ce-42c0e1fadb1d/c35708e6-dbe6-4af0-8b6b-22b8d851f6f1"
-					(reference "C31")
+					(reference "C11")
 					(unit 1)
 				)
@@
 		(dnp no)
 		(fields_autoplaced yes)
-		(property "Reference" "R24"
+		(property "Reference" "R29"
 			(at 140.97 86.3599 0)
 			(effects
@@
 			(project "microcard"
 				(path "/d4dbc2bb-914b-4f67-85ce-42c0e1fadb1d/c35708e6-dbe6-4af0-8b6b-22b8d851f6f1"
-					(reference "R24")
+					(reference "R29")
 					(unit 1)
 				)
@@
 		(dnp no)
 		(fields_autoplaced yes)
-		(property "Reference" "R26"
+		(property "Reference" "R32"
 			(at 74.93 93.9799 0)
 			(effects
@@
 			(project "microcard"
 				(path "/d4dbc2bb-914b-4f67-85ce-42c0e1fadb1d/c35708e6-dbe6-4af0-8b6b-22b8d851f6f1"
-					(reference "R26")
+					(reference "R32")
 					(unit 1)
 				)
@@
 		(dnp no)
 		(fields_autoplaced yes)
-		(property "Reference" "R33"
+		(property "Reference" "R26"
 			(at 74.93 80.0099 0)
 			(effects
@@
 			(project "microcard"
 				(path "/d4dbc2bb-914b-4f67-85ce-42c0e1fadb1d/c35708e6-dbe6-4af0-8b6b-22b8d851f6f1"
-					(reference "R33")
+					(reference "R26")
 					(unit 1)
 				)
@@
 		(dnp no)
 		(fields_autoplaced yes)
-		(property "Reference" "#PWR068"
+		(property "Reference" "#PWR045"
 			(at 138.43 87.63 0)
 			(effects
@@
 			(project ""
 				(path "/d4dbc2bb-914b-4f67-85ce-42c0e1fadb1d/c35708e6-dbe6-4af0-8b6b-22b8d851f6f1"
-					(reference "#PWR068")
+					(reference "#PWR045")
 					(unit 1)
 				)
@@
 		(dnp no)
 		(fields_autoplaced yes)
-		(property "Reference" "#PWR069"
+		(property "Reference" "#PWR048"
 			(at 97.79 82.55 0)
 			(effects
@@
 			(project "microcard"
 				(path "/d4dbc2bb-914b-4f67-85ce-42c0e1fadb1d/c35708e6-dbe6-4af0-8b6b-22b8d851f6f1"
-					(reference "#PWR069")
+					(reference "#PWR048")
 					(unit 1)
 				)
@@
 		(dnp no)
 		(fields_autoplaced yes)
-		(property "Reference" "R32"
+		(property "Reference" "R34"
 			(at 210.8201 101.6 0)
 			(effects
@@
 			(project "microcard"
 				(path "/d4dbc2bb-914b-4f67-85ce-42c0e1fadb1d/c35708e6-dbe6-4af0-8b6b-22b8d851f6f1"
-					(reference "R32")
+					(reference "R34")
 					(unit 1)
 				)
@@
 		(dnp no)
 		(fields_autoplaced yes)
-		(property "Reference" "#PWR078"
+		(property "Reference" "#PWR044"
 			(at 83.82 64.77 0)
 			(effects
@@
 			(project ""
 				(path "/d4dbc2bb-914b-4f67-85ce-42c0e1fadb1d/c35708e6-dbe6-4af0-8b6b-22b8d851f6f1"
-					(reference "#PWR078")
+					(reference "#PWR044")
 					(unit 1)
 				)
@@
 		(on_board yes)
 		(dnp no)
-		(property "Reference" "U8"
+		(property "Reference" "U5"
 			(at 88.9 96.266 0)
 			(effects
@@
 			(project ""
 				(path "/d4dbc2bb-914b-4f67-85ce-42c0e1fadb1d/c35708e6-dbe6-4af0-8b6b-22b8d851f6f1"
-					(reference "U8")
+					(reference "U5")
 					(unit 1)
 				)
@@
 		(on_board yes)
 		(dnp no)
-		(property "Reference" "#PWR077"
+		(property "Reference" "#PWR046"
 			(at 175.26 86.36 0)
 			(effects
@@
 			(project "microcard"
 				(path "/d4dbc2bb-914b-4f67-85ce-42c0e1fadb1d/c35708e6-dbe6-4af0-8b6b-22b8d851f6f1"
-					(reference "#PWR077")
+					(reference "#PWR046")
 					(unit 1)
 				)
@@
 		(on_board yes)
 		(dnp no)
-		(property "Reference" "LED1"
+		(property "Reference" "LED3"
 			(at 119.634 89.662 0)
 			(effects
@@
 			(project ""
 				(path "/d4dbc2bb-914b-4f67-85ce-42c0e1fadb1d/c35708e6-dbe6-4af0-8b6b-22b8d851f6f1"
-					(reference "LED1")
+					(reference "LED3")
 					(unit 1)
 				)
@@
 		(dnp no)
 		(fields_autoplaced yes)
-		(property "Reference" "Q6"
+		(property "Reference" "Q4"
 			(at 72.39 58.42 90)
 			(effects
@@
 			(project "microcard"
 				(path "/d4dbc2bb-914b-4f67-85ce-42c0e1fadb1d/c35708e6-dbe6-4af0-8b6b-22b8d851f6f1"
-					(reference "Q6")
+					(reference "Q4")
 					(unit 1)
 				)
@@
 		(on_board yes)
 		(dnp no)
-		(property "Reference" "LED3"
+		(property "Reference" "LED5"
 			(at 143.764 89.662 0)
 			(effects
@@
 			(project "microcard"
 				(path "/d4dbc2bb-914b-4f67-85ce-42c0e1fadb1d/c35708e6-dbe6-4af0-8b6b-22b8d851f6f1"
-					(reference "LED3")
+					(reference "LED5")
 					(unit 1)
 				)
@@
 		(dnp no)
 		(fields_autoplaced yes)
-		(property "Reference" "R29"
+		(property "Reference" "R31"
 			(at 173.99 88.8999 0)
 			(effects
@@
 			(project "microcard"
 				(path "/d4dbc2bb-914b-4f67-85ce-42c0e1fadb1d/c35708e6-dbe6-4af0-8b6b-22b8d851f6f1"
-					(reference "R29")
+					(reference "R31")
 					(unit 1)
 				)
@@
 		(dnp no)
 		(fields_autoplaced yes)
-		(property "Reference" "#PWR059"
+		(property "Reference" "#PWR047"
 			(at 80.01 82.55 0)
 			(effects
@@
 			(project ""
 				(path "/d4dbc2bb-914b-4f67-85ce-42c0e1fadb1d/c35708e6-dbe6-4af0-8b6b-22b8d851f6f1"
-					(reference "#PWR059")
+					(reference "#PWR047")
 					(unit 1)
 				)
@@
 		(dnp no)
 		(fields_autoplaced yes)
-		(property "Reference" "R25"
+		(property "Reference" "R30"
 			(at 152.4 86.3599 0)
 			(effects
@@
 			(project "microcard"
 				(path "/d4dbc2bb-914b-4f67-85ce-42c0e1fadb1d/c35708e6-dbe6-4af0-8b6b-22b8d851f6f1"
-					(reference "R25")
+					(reference "R30")
 					(unit 1)
 				)
@@
 		(dnp no)
 		(fields_autoplaced yes)
-		(property "Reference" "#PWR071"
+		(property "Reference" "#PWR049"
 			(at 105.41 90.17 0)
 			(effects
@@
 			(project "microcard"
 				(path "/d4dbc2bb-914b-4f67-85ce-42c0e1fadb1d/c35708e6-dbe6-4af0-8b6b-22b8d851f6f1"
-					(reference "#PWR071")
+					(reference "#PWR049")
 					(unit 1)
 				)
@@
 		(dnp no)
 		(fields_autoplaced yes)
-		(property "Reference" "D6"
+		(property "Reference" "D4"
 			(at 210.82 93.0274 90)
 			(effects
@@
 			(project "microcard"
 				(path "/d4dbc2bb-914b-4f67-85ce-42c0e1fadb1d/c35708e6-dbe6-4af0-8b6b-22b8d851f6f1"
-					(reference "D6")
+					(reference "D4")
 					(unit 1)
 				)
@@
 		(dnp no)
 		(fields_autoplaced yes)
-		(property "Reference" "Q3"
+		(property "Reference" "Q6"
 			(at 129.54 114.2999 0)
 			(effects
@@
 			(project "microcard"
 				(path "/d4dbc2bb-914b-4f67-85ce-42c0e1fadb1d/c35708e6-dbe6-4af0-8b6b-22b8d851f6f1"
-					(reference "Q3")
+					(reference "Q6")
 					(unit 1)
 				)
@@
 		(dnp no)
 		(fields_autoplaced yes)
-		(property "Reference" "R30"
+		(property "Reference" "R33"
 			(at 180.34 93.9799 0)
 			(effects
@@
 			(project "microcard"
 				(path "/d4dbc2bb-914b-4f67-85ce-42c0e1fadb1d/c35708e6-dbe6-4af0-8b6b-22b8d851f6f1"
-					(reference "R30")
+					(reference "R33")
 					(unit 1)
 				)
@@
 		(dnp no)
 		(fields_autoplaced yes)
-		(property "Reference" "R31"
+		(property "Reference" "R27"
 			(at 209.55 83.8199 0)
 			(effects
@@
 			(project "microcard"
 				(path "/d4dbc2bb-914b-4f67-85ce-42c0e1fadb1d/c35708e6-dbe6-4af0-8b6b-22b8d851f6f1"
-					(reference "R31")
+					(reference "R27")
 					(unit 1)
 				)
@@
 		(on_board yes)
 		(dnp no)
-		(property "Reference" "LED2"
+		(property "Reference" "LED4"
 			(at 132.334 89.662 0)
 			(effects
@@
 			(project "microcard"
 				(path "/d4dbc2bb-914b-4f67-85ce-42c0e1fadb1d/c35708e6-dbe6-4af0-8b6b-22b8d851f6f1"
-					(reference "LED2")
+					(reference "LED4")
 					(unit 1)
 				)
@@
 		(dnp no)
 		(fields_autoplaced yes)
-		(property "Reference" "R23"
+		(property "Reference" "R28"
 			(at 128.27 86.3599 0)
 			(effects
@@
 			(project ""
 				(path "/d4dbc2bb-914b-4f67-85ce-42c0e1fadb1d/c35708e6-dbe6-4af0-8b6b-22b8d851f6f1"
-					(reference "R23")
+					(reference "R28")
 					(unit 1)
 				)
@@
 		(dnp no)
 		(fields_autoplaced yes)
-		(property "Reference" "#PWR070"
+		(property "Reference" "#PWR050"
 			(at 125.73 127 0)
 			(effects
@@
 			(project "microcard"
 				(path "/d4dbc2bb-914b-4f67-85ce-42c0e1fadb1d/c35708e6-dbe6-4af0-8b6b-22b8d851f6f1"
-					(reference "#PWR070")
-					(unit 1)
-				)
+					(reference "#PWR050")
+					(unit 1)
+				)

Commit message: wide render
Parts:
- C11: footprint Capacitor_SMD:C_0603_1608Metric_Pad1.08x0.95mm_HandSolder -> Capacitor_SMD:C_0603_1608Metric
- D4, D5: footprint Diode_SMD:D_0603_1608Metric_Pad1.05x0.95mm_HandSolder -> Diode_SMD:D_0603Metric
- R26, R27, R28, R29, R30, R31, R32, R33, R34: footprint Resistor_SMD:R_0603_1608Metric_Pad0.98x0.95mm_HandSolder -> Resistor_SMD:R_0603_1608Metric
Changed lines of the file:
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@@
 			)
 		)
-		(property "Footprint" "Capacitor_SMD:C_0603_1608Metric_Pad1.08x0.95mm_HandSolder"
+		(property "Footprint" "Capacitor_SMD:C_0603_1608Metric"
 			(at 105.41 91.44 0)
 			(effects
@@
 			)
 		)
-		(property "Footprint" "Diode_SMD:D_0603_1608Metric_Pad1.05x0.95mm_HandSolder"
+		(property "Footprint" "Diode_SMD:D_0603Metric"
 			(at 171.45 97.79 0)
 			(effects
@@
 			)
 		)
-		(property "Footprint" "Resistor_SMD:R_0603_1608Metric_Pad0.98x0.95mm_HandSolder"
+		(property "Footprint" "Resistor_SMD:R_0603_1608Metric"
 			(at 136.652 87.63 90)
 			(effects
@@
 			)
 		)
-		(property "Footprint" "Resistor_SMD:R_0603_1608Metric_Pad0.98x0.95mm_HandSolder"
+		(property "Footprint" "Resistor_SMD:R_0603_1608Metric"
 			(at 74.168 95.25 90)
 			(effects
@@
 			)
 		)
-		(property "Footprint" "Resistor_SMD:R_0603_1608Metric_Pad0.98x0.95mm_HandSolder"
+		(property "Footprint" "Resistor_SMD:R_0603_1608Metric"
 			(at 74.168 81.28 90)
 			(effects
@@
 			)
 		)
-		(property "Footprint" "Resistor_SMD:R_0603_1608Metric_Pad0.98x0.95mm_HandSolder"
+		(property "Footprint" "Resistor_SMD:R_0603_1608Metric"
 			(at 209.55 100.838 90)
 			(effects
@@
 			)
 		)
-		(property "Footprint" "Resistor_SMD:R_0603_1608Metric_Pad0.98x0.95mm_HandSolder"
+		(property "Footprint" "Resistor_SMD:R_0603_1608Metric"
 			(at 173.228 90.17 90)
 			(effects
@@
 			)
 		)
-		(property "Footprint" "Resistor_SMD:R_0603_1608Metric_Pad0.98x0.95mm_HandSolder"
+		(property "Footprint" "Resistor_SMD:R_0603_1608Metric"
 			(at 148.082 87.63 90)
 			(effects
@@
 			)
 		)
-		(property "Footprint" "Diode_SMD:D_0603_1608Metric_Pad1.05x0.95mm_HandSolder"
+		(property "Footprint" "Diode_SMD:D_0603Metric"
 			(at 207.01 92.71 0)
 			(effects
@@
 			)
 		)
-		(property "Footprint" "Resistor_SMD:R_0603_1608Metric_Pad0.98x0.95mm_HandSolder"
+		(property "Footprint" "Resistor_SMD:R_0603_1608Metric"
 			(at 179.578 95.25 90)
 			(effects
@@
 			)
 		)
-		(property "Footprint" "Resistor_SMD:R_0603_1608Metric_Pad0.98x0.95mm_HandSolder"
+		(property "Footprint" "Resistor_SMD:R_0603_1608Metric"
 			(at 208.788 85.09 90)
 			(effects
@@
 			)
 		)
-		(property "Footprint" "Resistor_SMD:R_0603_1608Metric_Pad0.98x0.95mm_HandSolder"
+		(property "Footprint" "Resistor_SMD:R_0603_1608Metric"
 			(at 123.952 87.63 90)
 			(effects
