File: microcard/microcard.kicad_pcb (KiCad board)
At the start: 2 copper layers, 173.2 x 54 mm, 137 parts, among them CN1 CONMHF4-SMD-G-T, CN2 HC-1.2-4PWT, J1 Conn_01x08, J2 CHG, J3 BAT, Q1 BSS138PS,115, Q2 2N7002, Q3 2N7002, Q4 2N7002, Q5 BSS138PS,115, Q6 2N7002, Q7 2N7002, SW1 BOOT, SW2 RST, SW3 DIM, SW4 POW, SW5 SEL, SW6 ESC, SW7 UP, SW8 DWN, SW9 TRG, U1 ESP32-WROOM-32UE, U2 BQ24090DGQ, U3 TPS73633DBV, U4 ST25R3916-AQWT, U7 ADS1110, U8 DYWH-IRM-H238T/2T, X2 XRCGB27M120F3M00R0

Commit message: semi-finished pcb, pages
Parts:
- added AE1_FoldPads: , , F.SilkS at (184.5, 80.0)
- J3: footprint Connector_PinHeader_2.00mm:PinHeader_1x02_P2.00mm_Vertical -> Foldable:LiPo_302025
- moved SW9 124.7 mm to (153.0, 120.3)
- moved C40 95.2 mm to (119.4, 179.5)
- moved JP2 95.2 mm to (114.8, 176.6)
- moved TP2 95.2 mm to (140.7, 149.8)
- moved C41 95.2 mm to (110.5, 177.6)
- moved C43 95.2 mm to (110.5, 180.1)
- moved C44 95.2 mm to (120.0, 176.3)
- moved D6 95.2 mm to (144.9, 150.4)
- moved JP1 95.2 mm to (114.8, 173.1)
- moved Q7 95.2 mm to (145.1, 146.2)
- moved RV1 95.2 mm to (152.0, 156.4)
- moved TP1 95.2 mm to (140.7, 145.8)
- moved U6 95.2 mm to (135.0, 177.9)
- moved C39 95.2 mm to (110.5, 175.1)
- moved C42 95.2 mm to (120.0, 173.0)
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- renumbered ANT_2.54GHz1 to AE2, C44 to C1, C30 to C10, C31 to C11, C42 to C12, C33 to C13, C32 to C14, C43 to C15, C38 to C16, C34 to C17, C36 to C18, C18 to C19, C45 to C2, C19 to C20, C35 to C21, C37 to C22, C39 to C23, C16 to C24, C17 to C25, C28 to C26, C29 to C27, C24 to C28, C25 to C29, C1 to C3, C40 to C30, C26 to C31, C27 to C32, C20 to C33, C21 to C34, C41 to C35, C22 to C36, C23 to C37, C8 to C38, C9 to C39, C2 to C4, C10 to C40, C11 to C41, C12 to C42, C13 to C43, C14 to C44, C15 to C45, C3 to C5, C4 to C6, C5 to C7, C6 to C8, C7 to C9, CN2 to CN1, CN1 to CN2, D6 to D4, D4 to D6, L3 to L1, L4 to L2, L1 to L3, L2 to L4, LED4 to LED1, LED5 to LED2, LED1 to LED3, LED2 to LED4, LED3 to LED5, Q7 to Q1, Q1 to Q2, Q4 to Q3, Q6 to Q4, Q3 to Q6, Q2 to Q7, R38 to R10, R2 to R11, R3 to R12, R6 to R13, R8 to R14, R9 to R15, R4 to R16, R10 to R17, R7 to R18, R5 to R19, R40 to R2, R18 to R20, R16 to R21, R11 to R22, R19 to R23, R12 to R24, R20 to R25, R33 to R26, R31 to R27, R23 to R28, R24 to R29, R39 to R3, R25 to R30, R29 to R31, R26 to R32, R30 to R33, R32 to R34, R21 to R35, R22 to R36, R14 to R37, R15 to R38, R13 to R39, R28 to R4, R17 to R40, R27 to R5, R34 to R6, R35 to R7, R36 to R8, R37 to R9, SW5 to SW2, SW6 to SW3, SW7 to SW4, SW8 to SW5, SW9 to SW6, SW3 to SW7, SW2 to SW8, SW4 to SW9, U7 to U4, U8 to U5, U4 to U6, X2 to X1
Routing:
- net Net-(C45-Pad1): track 0.00 -> 3.36 mm
- net Net-(C45-Pad2): track 0.00 -> 3.10 mm
- added copper zone on F.Cu, net GND
Other:
- board size 173.2 x 54 mm -> 173.2 x 128.4 mm
- board text added: "U6"
- board text removed: "U4"

Commit message: wide render
Parts:
- removed AE1_FoldPads: , 
- added J2_FoldPads: , , F.SilkS at (55.6, 87.8)
- C1, C11, C13, C14, C2, C20, C25, C27, C29, C32, C34, C37, C38, C39, C4, C41, C43, C9: footprint Capacitor_SMD:C_0603_1608Metric_Pad1.08x0.95mm_HandSolder -> Capacitor_SMD:C_0603_1608Metric
- C10, C3, C40, C5, C6, C7, C8: footprint Capacitor_SMD:C_0805_2012Metric_Pad1.18x1.45mm_HandSolder -> Capacitor_SMD:C_0805_2012Metric
- C12, C15, C16, C17, C18, C21, C22, C23, C30, C35, C45: footprint Capacitor_SMD:C_0603_1608Metric_Pad1.08x0.95mm_HandSolder -> Capacitor_SMD:C_0402_1005Metric
- C19, C24, C26, C28, C31, C33, C36: footprint Capacitor_SMD:C_0402_1005Metric_Pad0.74x0.62mm_HandSolder -> Capacitor_SMD:C_0402_1005Metric
- C42, C44: footprint Capacitor_SMD:C_1206_3216Metric_Pad1.33x1.80mm_HandSolder -> Capacitor_SMD:C_1206_3216Metric
- L1, L2, L3, L4: footprint Inductor_SMD:L_0603_1608Metric_Pad1.05x0.95mm_HandSolder -> Inductor_SMD:L_0402_1005Metric
- R1, R10, R11, R12, R13, R14, R15, R16, R17, R18, R19, R20, R21, R22, R23, R24, R25, R26, R27, R28, R29, R3, R30, R31, R32, R33, R34, R35, R36, R37, R38, R39, R4, R40, R5, R6, R7, R8, R9: footprint Resistor_SMD:R_0603_1608Metric_Pad0.98x0.95mm_HandSolder -> Resistor_SMD:R_0603_1608Metric
- R2: footprint Resistor_SMD:R_0805_2012Metric_Pad1.20x1.40mm_HandSolder -> Resistor_SMD:R_0805_2012Metric
- moved D2 144.9 mm to (156.3, 163.4)
- moved LED4 144.9 mm to (154.8, 133.5)
- moved C1 144.9 mm to (129.3, 129.1)
- moved C10 144.9 mm to (156.5, 168.8)
- moved C14 144.9 mm to (128.5, 157.4)
- moved C20 144.9 mm to (124.1, 159.9)
- moved C25 144.9 mm to (124.1, 157.4)
- moved C27 144.9 mm to (124.1, 172.4)
- moved C29 144.9 mm to (124.1, 167.4)
- moved C37 144.9 mm to (124.1, 164.9)
- moved C9 144.9 mm to (146.8, 157.4)
- moved CN1 144.9 mm to (139.7, 135.9)
- moved D3 144.9 mm to (156.3, 166.0)
- moved LED3 144.9 mm to (154.8, 130.1)
- moved LED5 144.9 mm to (154.8, 137.0)
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Routing:
- net Net-(C45-Pad2): track 3.10 -> 5.34 mm
- net Net-(C45-Pad1): track 3.36 -> 2.05 mm
- net Net-(AE2-FEED): track 0.00 -> 0.94 mm
Other:
- board size 173.2 x 128.4 mm -> 173.2 x 54 mm
- board text added: "CHG"
