File: microcard/microcard.kicad_sch (KiCad schematic)
At the start: 32 parts, among them CN2 HC-1.2-4PWT, J1 Conn_01x08, J2 CHG, Q7 2N7002, SW1 BOOT, SW2 RST, SW3 DIM, SW5 SEL, SW6 ESC, SW7 UP, SW8 DWN, SW9 TRG, U1 ESP32-WROOM-32UE

Commit message: semi-finished pcb, pages
Parts:
- renumbered C44 to C1, C45 to C2, C1 to C3, C2 to C4, CN2 to CN1, LED4 to LED1, LED5 to LED2, Q7 to Q1, R38 to R10, R2 to R11, R3 to R12, R40 to R2, R39 to R3, R28 to R4, R27 to R5, R34 to R6, R35 to R7, R36 to R8, R37 to R9, SW5 to SW2, SW6 to SW3, SW7 to SW4, SW8 to SW5, SW9 to SW6, SW3 to SW7, SW2 to SW8

Commit message: wide render
Parts:
- C1, C2, C4: footprint Capacitor_SMD:C_0603_1608Metric_Pad1.08x0.95mm_HandSolder -> Capacitor_SMD:C_0603_1608Metric
- C3: footprint Capacitor_SMD:C_0805_2012Metric_Pad1.18x1.45mm_HandSolder -> Capacitor_SMD:C_0805_2012Metric
- D1: footprint Diode_SMD:D_0603_1608Metric_Pad1.05x0.95mm_HandSolder -> Diode_SMD:D_0603Metric
- R1, R10, R11, R12, R3, R4, R5, R6, R7, R8, R9: footprint Resistor_SMD:R_0603_1608Metric_Pad0.98x0.95mm_HandSolder -> Resistor_SMD:R_0603_1608Metric
- R2: footprint Resistor_SMD:R_0805_2012Metric_Pad1.20x1.40mm_HandSolder -> Resistor_SMD:R_0805_2012Metric
Other:
- moved on the sheet: C1, C2, C3, C4, CN1, D1, J1, J2, LED1, LED2, Q1, R1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
