File: microcard/nfc_rfid.kicad_sch (KiCad schematic)
At the start: 39 parts, among them Q2 2N7002, U4 ST25R3916-AQWT, X2 XRCGB27M120F3M00R0

Commit message: semi-finished pcb, pages
Parts:
- renumbered C42 to C12, C33 to C13, C32 to C14, C43 to C15, C38 to C16, C34 to C17, C36 to C18, C18 to C19, C19 to C20, C35 to C21, C37 to C22, C39 to C23, C16 to C24, C17 to C25, C28 to C26, C29 to C27, C24 to C28, C25 to C29, C40 to C30, C26 to C31, C27 to C32, C20 to C33, C21 to C34, C41 to C35, C22 to C36, C23 to C37, D4 to D6, L3 to L1, L4 to L2, Q2 to Q7, R21 to R35, R22 to R36, R14 to R37, R15 to R38, U4 to U6, X2 to X1

Commit message: wide render
Parts:
- C12, C15, C16, C17, C18, C21, C22, C23, C30, C35: footprint Capacitor_SMD:C_0603_1608Metric_Pad1.08x0.95mm_HandSolder -> Capacitor_SMD:C_0402_1005Metric
- C13, C14, C20, C25, C27, C29, C32, C34, C37: footprint Capacitor_SMD:C_0603_1608Metric_Pad1.08x0.95mm_HandSolder -> Capacitor_SMD:C_0603_1608Metric
- C19, C24, C26, C28, C31, C33, C36: footprint Capacitor_SMD:C_0402_1005Metric_Pad0.74x0.62mm_HandSolder -> Capacitor_SMD:C_0402_1005Metric
- L1, L2: footprint Inductor_SMD:L_0603_1608Metric_Pad1.05x0.95mm_HandSolder -> Inductor_SMD:L_0402_1005Metric
- R35, R36, R37, R38: footprint Resistor_SMD:R_0603_1608Metric_Pad0.98x0.95mm_HandSolder -> Resistor_SMD:R_0603_1608Metric
Other:
- moved on the sheet: AE1, C12, C13, C14, C15, C16, C17, C18, C19, C20, C21, C22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
