File: microcard/oled_sd1315.kicad_sch (KiCad schematic)
At the start: 13 parts, among them J4 OLED_SSD1315

Commit message: semi-finished pcb, pages
Parts:
- renumbered C8 to C38, C9 to C39, C10 to C40, C11 to C41, C12 to C42, C13 to C43, C14 to C44, R13 to R39, R17 to R40
Changed lines of the file:
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@@
 		(dnp no)
 		(fields_autoplaced yes)
-		(property "Reference" "R13"
+		(property "Reference" "R39"
 			(at 93.98 87.6299 0)
 			(effects
@@
 			(project ""
 				(path "/d4dbc2bb-914b-4f67-85ce-42c0e1fadb1d/d6a241b9-3d6e-4052-950a-687333676ee3"
-					(reference "R13")
+					(reference "R39")
 					(unit 1)
 				)
@@
 		(dnp no)
 		(fields_autoplaced yes)
-		(property "Reference" "#PWR054"
+		(property "Reference" "#PWR078"
 			(at 160.02 62.23 0)
 			(effects
@@
 			(project ""
 				(path "/d4dbc2bb-914b-4f67-85ce-42c0e1fadb1d/d6a241b9-3d6e-4052-950a-687333676ee3"
-					(reference "#PWR054")
+					(reference "#PWR078")
 					(unit 1)
 				)
@@
 		(dnp no)
 		(fields_autoplaced yes)
-		(property "Reference" "#PWR057"
+		(property "Reference" "#PWR076"
 			(at 172.72 33.02 0)
 			(effects
@@
 			(project ""
 				(path "/d4dbc2bb-914b-4f67-85ce-42c0e1fadb1d/d6a241b9-3d6e-4052-950a-687333676ee3"
-					(reference "#PWR057")
+					(reference "#PWR076")
 					(unit 1)
 				)
@@
 		(dnp no)
 		(fields_autoplaced yes)
-		(property "Reference" "#PWR058"
+		(property "Reference" "#PWR082"
 			(at 172.72 119.38 0)
 			(effects
@@
 			(project ""
 				(path "/d4dbc2bb-914b-4f67-85ce-42c0e1fadb1d/d6a241b9-3d6e-4052-950a-687333676ee3"
-					(reference "#PWR058")
+					(reference "#PWR082")
 					(unit 1)
 				)
@@
 		(dnp no)
 		(fields_autoplaced yes)
-		(property "Reference" "#PWR037"
+		(property "Reference" "#PWR081"
 			(at 91.44 104.14 0)
 			(effects
@@
 			(project ""
 				(path "/d4dbc2bb-914b-4f67-85ce-42c0e1fadb1d/d6a241b9-3d6e-4052-950a-687333676ee3"
-					(reference "#PWR037")
+					(reference "#PWR081")
 					(unit 1)
 				)
@@
 		(on_board yes)
 		(dnp no)
-		(property "Reference" "C12"
+		(property "Reference" "C42"
 			(at 112.268 96.012 0)
 			(effects
@@
 			(project ""
 				(path "/d4dbc2bb-914b-4f67-85ce-42c0e1fadb1d/d6a241b9-3d6e-4052-950a-687333676ee3"
-					(reference "C12")
+					(reference "C42")
 					(unit 1)
 				)
@@
 		(on_board yes)
 		(dnp no)
-		(property "Reference" "C14"
+		(property "Reference" "C44"
 			(at 125.73 96.012 0)
 			(effects
@@
 			(project ""
 				(path "/d4dbc2bb-914b-4f67-85ce-42c0e1fadb1d/d6a241b9-3d6e-4052-950a-687333676ee3"
-					(reference "C14")
+					(reference "C44")
 					(unit 1)
 				)
@@
 		(dnp no)
 		(fields_autoplaced yes)
-		(property "Reference" "#PWR038"
+		(property "Reference" "#PWR083"
 			(at 138.43 142.24 0)
 			(effects
@@
 			(project ""
 				(path "/d4dbc2bb-914b-4f67-85ce-42c0e1fadb1d/d6a241b9-3d6e-4052-950a-687333676ee3"
-					(reference "#PWR038")
+					(reference "#PWR083")
 					(unit 1)
 				)
@@
 		(dnp no)
 		(fields_autoplaced yes)
-		(property "Reference" "#PWR036"
+		(property "Reference" "#PWR077"
 			(at 101.6 66.04 0)
 			(effects
@@
 			(project ""
 				(path "/d4dbc2bb-914b-4f67-85ce-42c0e1fadb1d/d6a241b9-3d6e-4052-950a-687333676ee3"
-					(reference "#PWR036")
+					(reference "#PWR077")
 					(unit 1)
 				)
@@
 		(on_board yes)
 		(dnp no)
-		(property "Reference" "C13"
+		(property "Reference" "C43"
 			(at 119.888 96.012 0)
 			(effects
@@
 			(project ""
 				(path "/d4dbc2bb-914b-4f67-85ce-42c0e1fadb1d/d6a241b9-3d6e-4052-950a-687333676ee3"
-					(reference "C13")
+					(reference "C43")
 					(unit 1)
 				)
@@
 		(on_board yes)
 		(dnp no)
-		(property "Reference" "C11"
+		(property "Reference" "C41"
 			(at 107.188 96.012 0)
 			(effects
@@
 			(project ""
 				(path "/d4dbc2bb-914b-4f67-85ce-42c0e1fadb1d/d6a241b9-3d6e-4052-950a-687333676ee3"
-					(reference "C11")
+					(reference "C41")
 					(unit 1)
 				)
@@
 		(on_board yes)
 		(dnp no)
-		(property "Reference" "C9"
+		(property "Reference" "C39"
 			(at 119.38 40.386 0)
 			(effects
@@
 			(project ""
 				(path "/d4dbc2bb-914b-4f67-85ce-42c0e1fadb1d/d6a241b9-3d6e-4052-950a-687333676ee3"
-					(reference "C9")
+					(reference "C39")
 					(unit 1)
 				)
@@
 		(on_board yes)
 		(dnp no)
-		(property "Reference" "C8"
+		(property "Reference" "C38"
 			(at 91.186 40.386 0)
 			(effects
@@
 			(project ""
 				(path "/d4dbc2bb-914b-4f67-85ce-42c0e1fadb1d/d6a241b9-3d6e-4052-950a-687333676ee3"
-					(reference "C8")
+					(reference "C38")
 					(unit 1)
 				)
@@
 		(dnp no)
 		(fields_autoplaced yes)
-		(property "Reference" "#PWR056"
+		(property "Reference" "#PWR080"
 			(at 160.02 67.31 0)
 			(effects
@@
 			(project ""
 				(path "/d4dbc2bb-914b-4f67-85ce-42c0e1fadb1d/d6a241b9-3d6e-4052-950a-687333676ee3"
-					(reference "#PWR056")
+					(reference "#PWR080")
 					(unit 1)
 				)
@@
 		(dnp no)
 		(fields_autoplaced yes)
-		(property "Reference" "#PWR055"
+		(property "Reference" "#PWR079"
 			(at 170.18 64.77 0)
 			(effects
@@
 			(project ""
 				(path "/d4dbc2bb-914b-4f67-85ce-42c0e1fadb1d/d6a241b9-3d6e-4052-950a-687333676ee3"
-					(reference "#PWR055")
+					(reference "#PWR079")
 					(unit 1)
 				)
@@
 		(dnp no)
 		(fields_autoplaced yes)
-		(property "Reference" "R17"
+		(property "Reference" "R40"
 			(at 170.18 130.8099 0)
 			(effects
@@
 			(project ""
 				(path "/d4dbc2bb-914b-4f67-85ce-42c0e1fadb1d/d6a241b9-3d6e-4052-950a-687333676ee3"
-					(reference "R17")
+					(reference "R40")
 					(unit 1)
 				)
@@
 		(dnp no)
 		(fields_autoplaced yes)
-		(property "Reference" "#PWR053"
+		(property "Reference" "#PWR084"
 			(at 167.64 142.24 0)
 			(effects
@@
 			(project ""
 				(path "/d4dbc2bb-914b-4f67-85ce-42c0e1fadb1d/d6a241b9-3d6e-4052-950a-687333676ee3"
-					(reference "#PWR053")
+					(reference "#PWR084")
 					(unit 1)
 				)
@@
 		(on_board yes)
 		(dnp no)
-		(property "Reference" "C10"
+		(property "Reference" "C40"
 			(at 95.504 95.758 0)
 			(effects
@@
 			(project ""
 				(path "/d4dbc2bb-914b-4f67-85ce-42c0e1fadb1d/d6a241b9-3d6e-4052-950a-687333676ee3"
-					(reference "C10")
-					(unit 1)
-				)
+					(reference "C40")
+					(unit 1)
+				)

Commit message: wide render
Parts:
- C38, C39, C41, C43: footprint Capacitor_SMD:C_0603_1608Metric_Pad1.08x0.95mm_HandSolder -> Capacitor_SMD:C_0603_1608Metric
- C40: footprint Capacitor_SMD:C_0805_2012Metric_Pad1.18x1.45mm_HandSolder -> Capacitor_SMD:C_0805_2012Metric
- C42, C44: footprint Capacitor_SMD:C_1206_3216Metric_Pad1.33x1.80mm_HandSolder -> Capacitor_SMD:C_1206_3216Metric
- R39, R40: footprint Resistor_SMD:R_0603_1608Metric_Pad0.98x0.95mm_HandSolder -> Resistor_SMD:R_0603_1608Metric
Other:
- moved on the sheet: J4
